File: Board/waterius-homemade.brd (EAGLE design)
At the start: 13.5 x 60 mm, 24 parts, among them IC1 TINY13-20SU

Commit message: инструкция, плата для производства
Parts:
- removed R11: 300, rcl:R0805
- LED1: device led:SML0805 -> led:LED3MM
- R10: value 0 -> 300
- R4: device rcl:0207/2V -> rcl:R0805
- moved R10 11.4 mm to (11.1, 32.4)
- moved RST 2.63 mm to (10.7, 38.1)
- moved R8 2.45 mm to (8.13, 31.3)
- moved R1 2.15 mm to (6.64, 44.1), turned to 0 degrees
- moved C7 1.66 mm to (9.24, 35.6), turned to 180 degrees
- moved C4 1.66 mm to (9.21, 29.4), turned to 0 degrees
- moved R6 1.46 mm to (9.72, 48.3), turned to 0 degrees
- moved C1 0.79 mm to (6.35, 4.16)
- moved JP1 0.64 mm to (10.6, 4.32)
- moved R3 0.48 mm to (3.27, 24.1)
- moved R7 0.48 mm to (3.27, 21.4)
- moved LED1 0.39 mm to (10.9, 9.91), turned to 270 degrees
- moved R2 0.33 mm to (8.06, 24.1)
- moved C2 0.22 mm to (2.67, 8.64)
- moved R4 0.22 mm to (7.27, 8.67)
Connections:
- removed net N$2: R11.1, S2.1
- net GND1: now also S2.1; no longer R11.2
- net N$6: now also LED1.K; no longer LED1.C
Routing:
- net GND1: track 45.8 -> 36.7 mm
- net N$2: track 6.02 -> 0.00 mm
- net +3V3: track 41.4 -> 44.6 mm
- net N$4: track 16.2 -> 13.3 mm
- net IN1: track 14.4 -> 16.2 mm
- net IN2: track 10.0 -> 11.7 mm
- net GND: track 58.3 -> 59.8 mm
- net N$3: track 5.00 -> 4.11 mm
- net AA*3: track 8.00 -> 8.68 mm
