File: Board/waterius-homemade.sch (EAGLE design)
At the start: 24 parts, among them IC1 TINY13-20SU

Commit message: инструкция, плата для производства
Parts:
- removed R11: 300, rcl:R-EU_R0805
- LED1: device led:LEDSML0805 -> led:LED3MM
- R10: value 0 -> 300
- R4: device rcl:R-EU_0207/2V -> rcl:R-EU_R0805
Connections:
- removed net N$2: R11.1, S2.P
- net GND1: now also S2.P; no longer R11.2
