File: Board/waterius-factory-2.0.brd (EAGLE design)
At the start: 13.5 x 51 mm, 23 parts, among them IC1 TINY85-20SU, U3 ESP01

Commit message: correct board
Parts:
- flipped JP1 to the bottom, turned to 270 degrees
- flipped LOG to the bottom
Routing:
- net GND: track 50.8 -> 51.4 mm
- net SCK: vias 2 -> 1
- net GND1: vias 1 -> 0
Changed lines of the file:
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@@
 <drawing>
 <settings>
-<setting alwaysvectorfont="no"/>
+<setting alwaysvectorfont="yes"/>
 <setting keepoldvectorfont="yes"/>
 <setting verticaltext="up"/>
@@
 <layer number="16" name="Bottom" color="1" fill="1" visible="yes" active="yes"/>
 <layer number="17" name="Pads" color="2" fill="1" visible="yes" active="yes"/>
-<layer number="18" name="Vias" color="2" fill="1" visible="no" active="yes"/>
+<layer number="18" name="Vias" color="2" fill="1" visible="yes" active="yes"/>
 <layer number="19" name="Unrouted" color="6" fill="1" visible="yes" active="yes"/>
-<layer number="20" name="Dimension" color="24" fill="1" visible="no" active="yes"/>
-<layer number="21" name="tPlace" color="7" fill="1" visible="no" active="yes"/>
-<layer number="22" name="bPlace" color="7" fill="1" visible="no" active="yes"/>
+<layer number="20" name="Dimension" color="24" fill="1" visible="yes" active="yes"/>
+<layer number="21" name="tPlace" color="7" fill="1" visible="yes" active="yes"/>
+<layer number="22" name="bPlace" color="7" fill="1" visible="yes" active="yes"/>
 <layer number="23" name="tOrigins" color="15" fill="1" visible="yes" active="yes"/>
 <layer number="24" name="bOrigins" color="15" fill="1" visible="yes" active="yes"/>
 <layer number="25" name="tNames" color="7" fill="1" visible="yes" active="yes"/>
-<layer number="26" name="bNames" color="7" fill="1" visible="no" active="yes"/>
-<layer number="27" name="tValues" color="7" fill="1" visible="no" active="yes"/>
-<layer number="28" name="bValues" color="7" fill="1" visible="no" active="yes"/>
+<layer number="26" name="bNames" color="7" fill="1" visible="yes" active="yes"/>
+<layer number="27" name="tValues" color="7" fill="1" visible="yes" active="yes"/>
+<layer number="28" name="bValues" color="7" fill="1" visible="yes" active="yes"/>
 <layer number="29" name="tStop" color="7" fill="3" visible="no" active="yes"/>
 <layer number="30" name="bStop" color="7" fill="6" visible="no" active="yes"/>
@@
 <layer number="38" name="bTest" color="7" fill="1" visible="no" active="yes"/>
 <layer number="39" name="tKeepout" color="4" fill="11" visible="yes" active="yes"/>
-<layer number="40" name="bKeepout" color="1" fill="11" visible="no" active="yes"/>
+<layer number="40" name="bKeepout" color="1" fill="11" visible="yes" active="yes"/>
 <layer number="41" name="tRestrict" color="4" fill="10" visible="yes" active="yes"/>
-<layer number="42" name="bRestrict" color="1" fill="10" visible="no" active="yes"/>
+<layer number="42" name="bRestrict" color="1" fill="10" visible="yes" active="yes"/>
 <layer number="43" name="vRestrict" color="2" fill="10" visible="no" active="yes"/>
 <layer number="44" name="Drills" color="7" fill="1" visible="no" active="yes"/>
@@
 <layer number="49" name="Reference" color="7" fill="1" visible="no" active="yes"/>
 <layer number="51" name="tDocu" color="7" fill="1" visible="yes" active="yes"/>
-<layer number="52" name="bDocu" color="7" fill="1" visible="no" active="yes"/>
+<layer number="52" name="bDocu" color="7" fill="1" visible="yes" active="yes"/>
 <layer number="88" name="SimResults" color="9" fill="1" visible="no" active="no"/>
 <layer number="89" name="SimProbes" color="9" fill="1" visible="no" active="no"/>
@@
 <text x="12.2428" y="1.3" size="1" layer="26" rot="MR0">TX</text>
 <text x="1.8542" y="10.9982" size="1" layer="26" rot="MR270">waterius.ru</text>
-<text x="5.1562" y="8.001" size="1.5" layer="25">+</text>
+<text x="4.191" y="8.001" size="1.5" layer="25">+</text>
 <dimension x1="0" y1="0" x2="0" y2="7.5" x3="-10.774365625" y3="3.75" textsize="1.778" layer="47"/>
 <dimension x1="0" y1="0" x2="0" y2="30.5" x3="-15.66665" y3="15.25" textsize="1.778" layer="47"/>
-<text x="12.9286" y="35.3314" size="1.778" layer="26" rot="MR0">-   +</text>
+<text x="12.9286" y="35.3314" size="1.778" layer="26" rot="MR0">- +</text>
 <dimension x1="0" y1="52" x2="3.0226" y2="51.9684" x3="1.5338625" y3="54.1427" textsize="1.778" layer="1"/>
 <dimension x1="0" y1="0" x2="-0.0508" y2="39.5224" x3="-11.58323125" y3="19.74634375" textsize="1.778" layer="1"/>
 <text x="1.8542" y="14.4018" size="1" layer="26" rot="MR270">v0.2</text>
 <text x="9.3218" y="1.3" size="1" layer="26" rot="MR0">EN</text>
-<text x="6.477" y="5.461" size="1.5" layer="26" rot="MR0">+</text>
-<text x="8.8138" y="35.2044" size="1.778" layer="25">+  -</text>
+<text x="5.3848" y="8.0264" size="1.5" layer="26" rot="MR0">+</text>
+<text x="8.5598" y="35.306" size="1.778" layer="25">+  -</text>
 <wire x1="1.6256" y1="2.6924" x2="13.0556" y2="2.6924" width="0.1016" layer="26"/>
 <wire x1="4.5212" y1="4.2" x2="4.5212" y2="1" width="0.1016" layer="26"/>
@@
 </autorouter>
 <elements>
-<element name="JP1" library="jumper" package="JP1" value="" x="10.907" y="33.7976" smashed="yes" rot="R90">
-<attribute name="VALUE" x="12.5326" y="36.49" size="1.27" layer="27" ratio="10" rot="R180"/>
+<element name="JP1" library="jumper" package="JP1" value="" x="10.907" y="33.7976" smashed="yes" rot="MR270">
+<attribute name="VALUE" x="12.5326" y="31.1052" size="1.27" layer="28" ratio="10" rot="MR0"/>
 </element>
 <element name="C1" library="rcl" package="C0805" value="1uF" x="11.2254" y="30.4868" smashed="yes" rot="MR180">
@@
 <attribute name="NAME" x="11.3596" y="47.4668" size="1" layer="25"/>
 </element>
-<element name="LOG" library="pinhead" package="1X01" value="" x="10.0348" y="8.7476" smashed="yes">
-<attribute name="NAME" x="11.8452" y="7.1898" size="1" layer="26" ratio="10" rot="MR90"/>
-<attribute name="VALUE" x="8.7648" y="5.5726" size="1.27" layer="27"/>
+<element name="LOG" library="pinhead" package="1X01" value="" x="10.0348" y="8.7476" smashed="yes" rot="MR0">
+<attribute name="NAME" x="8.2244" y="7.1898" size="1" layer="25" ratio="10" rot="R90"/>
+<attribute name="VALUE" x="11.3048" y="5.5726" size="1.27" layer="28" rot="MR0"/>
 </element>
 <element name="R3" library="resistor" package="R0805" value="300" x="8.6498" y="30.0664" smashed="yes">
@@
 <contactref element="C1" pad="1"/>
 <contactref element="U$1" pad="3"/>
-<wire x1="9.637" y1="33.7976" x2="9.637" y2="31.303" width="0.3048" layer="16"/>
-<wire x1="9.637" y1="31.303" x2="10.2754" y2="30.4868" width="0.3048" layer="16"/>
 <wire x1="10.2754" y1="30.4868" x2="9.6404" y2="29.7572" width="0.3048" layer="16"/>
 <wire x1="9.6404" y1="29.7572" x2="9.6266" y2="27.432" width="0.3048" layer="16"/>
 <wire x1="9.6266" y1="27.432" x2="9.398" y2="27.3812" width="0.3048" layer="16"/>
+<wire x1="10.2754" y1="30.4868" x2="9.637" y2="31.1252" width="0.3048" layer="16"/>
+<wire x1="9.637" y1="31.1252" x2="9.637" y2="33.7976" width="0.3048" layer="16"/>
 </signal>
 <signal name="+3V">
@@
 <wire x1="10.2616" y1="37.0332" x2="11.4808" y2="38.2524" width="0.3048" layer="16"/>
 <wire x1="3.6068" y1="37.0332" x2="10.2616" y2="37.0332" width="0.3048" layer="16"/>
-<via x="5.4392" y="30.07" extent="1-16" drill="0.35"/>
 <contactref element="S1" pad="2"/>
-<wire x1="5.4392" y1="30.07" x2="2.8448" y2="32.6644" width="0.3048" layer="1"/>
-<wire x1="2.8448" y1="32.6644" x2="2.8194" y2="32.6644" width="0.3048" layer="1"/>
 <wire x1="2.8194" y1="32.6644" x2="2.8194" y2="36.195" width="0.3048" layer="16"/>
 <wire x1="2.8194" y1="36.195" x2="2.8448" y2="36.2204" width="0.3048" layer="16"/>
+<wire x1="2.8194" y1="32.6644" x2="2.8448" y2="32.6644" width="0.3048" layer="1"/>
+<wire x1="2.8448" y1="32.6644" x2="5.4392" y2="30.07" width="0.3048" layer="1"/>
 </signal>
 <signal name="N$7">
@@
 <wire x1="6.1038" y1="23.6298" x2="6.1038" y2="24.2566" width="0.3048" layer="16"/>
 <wire x1="5.3594" y1="22.8854" x2="6.1038" y2="23.6298" width="0.3048" layer="16"/>
-<wire x1="12.177" y1="33.7976" x2="12.177" y2="32.0698" width="0.3048" layer="16"/>
-<wire x1="12.177" y1="32.0698" x2="12.192" y2="31.0896" width="0.3048" layer="16"/>
 <wire x1="12.192" y1="31.0896" x2="12.192" y2="30.4018" width="0.3048" layer="16"/>
 <wire x1="12.192" y1="30.4018" x2="12.1754" y2="30.4868" width="0.3048" layer="16"/>
@@
 <wire x1="11.6586" y1="6.3246" x2="11.6586" y2="6.215" width="0.3048" layer="16"/>
 <wire x1="12.7" y1="12.4153" x2="11.2066" y2="13.9087" width="0.3048" layer="16"/>
+<wire x1="12.1754" y1="30.4868" x2="12.1754" y2="33.796" width="0.3048" layer="16"/>
+<wire x1="12.1754" y1="33.796" x2="12.177" y2="33.7976" width="0.3048" layer="16"/>
 </signal>
 <signal name="IN2">
@@
 <wire x1="8.4328" y1="20.828" x2="7.9248" y2="21.336" width="0.3048" layer="1"/>
 <wire x1="7.9248" y1="21.336" x2="7.5946" y2="21.6408" width="0.3048" layer="1"/>
-<via x="2.794" y="26.3906" extent="1-16" drill="0.35"/>
 <contactref element="S1" pad="1"/>
 <wire x1="2.794" y1="26.3906" x2="2.794" y2="28.1178" width="0.3048" layer="1"/>
@@
 <contactref element="LOG" pad="1"/>
 <contactref element="LED1" pad="A"/>
-<wire x1="10.0348" y1="8.7476" x2="10.795" y2="9.5078" width="0.3048" layer="1"/>
 <wire x1="10.795" y1="10.9571" x2="11.2066" y2="11.3687" width="0.3048" layer="1"/>
-<wire x1="10.795" y1="9.5078" x2="10.795" y2="10.9571" width="0.3048" layer="1"/>
-<wire x1="10.0348" y1="8.7476" x2="9.7434" y2="8.4562" width="0.3048" layer="1"/>
-<wire x1="10.0348" y1="8.7476" x2="7.381" y2="8.7354" width="0.3048" layer="1"/>
-<wire x1="7.381" y1="8.7354" x2="7.3424" y2="8.7354" width="0.3048" layer="1"/>
+<wire x1="10.0348" y1="8.7476" x2="7.3546" y2="8.7476" width="0.3048" layer="1"/>
+<wire x1="7.3546" y1="8.7476" x2="7.3424" y2="8.7354" width="0.3048" layer="1"/>
+<wire x1="10.0348" y1="8.7476" x2="10.0348" y2="10.1969" width="0.3048" layer="1"/>
+<wire x1="10.0348" y1="10.1969" x2="11.2066" y2="11.3687" width="0.3048" layer="1"/>
 </signal>
 <signal name="N$6">
