File: Board/waterius-factory-2.0wago.brd (EAGLE design)
At the start: 13.5 x 52 mm, 23 parts, among them IC1 TINY85-20SU, U3 ESP01, X2 235-104

Commit message: wago board update
Parts:
- moved R1 7.80 mm to (1.78, 37.1)
- moved R2 7.34 mm to (1.74, 44.7)
- flipped JP1 to the bottom, turned to 270 degrees
- flipped LOG to the bottom
- flipped R11 to the top, turned to 180 degrees
- flipped X2 to the bottom, turned to 0 degrees
Connections:
- removed net N$7: R1.1, X2.L3.1, X2.L3.2
- new net N$10: R1.1, X2.L4.1, X2.L4.2
- net GND1: now also X2.L1.1, X2.L1.2, X2.L3.1, X2.L3.2; no longer X2.L2.1, X2.L2.2, X2.L4.1, X2.L4.2
- net N$8: now also X2.L2.1, X2.L2.2; no longer X2.L1.1, X2.L1.2
Routing:
- net N$7: track 8.36 -> 0.00 mm
- net N$10: track 0.00 -> 8.26 mm
- net IN2: track 21.1 -> 28.7 mm, vias 1 -> 3
- net IN1: track 34.2 -> 27.0 mm
- net GND1: track 48.9 -> 44.2 mm
- net SCK: track 26.1 -> 26.0 mm, vias 2 -> 1
