File: Board/waterius-factory-3.0.sch (EAGLE design)
At the start: 24 parts, among them IC1 TINY13-20SU, U3 ESP01

Commit message: board v.0.3
Parts:
- removed PAD1: MOUNT-HOLE2.8, holes:MOUNT-HOLE2.8
- C2: value 1uF -> 0.1uF
- C4: value 0.1uF -> 1uF
- IC1: value TINY13-20SU -> TINY85-20SU
- JP1: value + - -> (none)
- R10, R3: value 3k3 -> 300
- R2, R8: value 300 -> 3k3
- U$1: device Microchip_By_element14_Batch_1:MCP1700T-3002E/TT -> MCP1700T-3002E_TT:MCP1700T-3002E/TT
Connections:
- net +3V: now also C4.1, R8.2, R9.2; no longer C3.1, R10.2, R4.2
- net GND: now also R10.1, R3.2, R4.1; no longer R2.2, R8.1, R9.1
- net GND1: now also R3.1, S1.S; no longer R2.1, S1.P
- net IN2: now also R2.2; no longer R3.2
- net N$2: now also R6.1; no longer R5.1
- net N$3: now also R9.1; no longer R4.1
- net N$4: now also C3.1, R5.1; no longer C4.1, R10.1
- net N$6: now also R10.2; no longer R8.2
- net N$8: now also R2.1; no longer R3.1
- net SCK: now also R8.1, S1.P; no longer R7.1, S1.S
- net SDA: now also R7.1; no longer R6.1
- net WAKE_UP: now also R4.2; no longer R9.2
Other:
- moved on the sheet: C3, C4, R10, R2, R3, R4, R5, R6, R7, R8, R9, S1
